Commit message: fix(asset): 修正左膝镜像轴方向并重建资产
现象：D2 的限位审计通过（25/25 一致），但运动学测试显示左右腿仍不对称。
定位：左膝 l_knee_y 的 axis 写的是 (0,0,-1)，右膝是 (0,0,1)。
      镜像关节要求"轴线同向 + 角度取反"（r = -l），左膝漏了符号翻转。

为什么这是"反关节站不稳"的真正嫌疑：
  膝盖是【单向】限位（右膝 [-2.339,+0.061]）。轴反向之后限位区间跟着镜像，
  物理上就允许膝盖朝反方向弯 —— RL 一定会找到这个作弊解。

修法：不对某条轴硬编码，而是对每一对镜像关节分别计算两种镜像约定下的
      可用运动窗口，只在"同号窗口 < 0.3 rad 且反号窗口 > 1.0 rad"时才翻转。
      这样只翻转真正可疑的 l_knee_y，不误伤 hip_x / hip_z
      （它们双向对称，翻转不改变物理，但会破坏 r = -l 这个干净约定，
        也会让后面所有基于镜像的推理变得可疑）。

验证：修正后 5 对镜像关节的足端位移完全对称；USD 重建后限位为
      l_knee_y [-0.061,+2.339] / r_knee_y [-2.339,+0.061]，严格镜像。

File: assets/poppy/urdf/Poppy_Humanoid_locked.urdf (robot description, URDF)
Before this commit: robot Poppy_Humanoid, 26 links, 25 joints
Joints:
- joint l_knee_y: axis 0 0 -1 -> 0 0 1
